Commit message: Relocate ai-models, update paths, full VLM training config, rewrite README
- Move ai-models/ from ~/lerobot/ to workspace root
- Update all hardcoded paths from /home/ubuntu/lerobot/ai-models to /home/ubuntu/ur3_ft300_ws/ai-models
- Add train_full_vlm.py for A100 full VLM fine-tuning (train_expert_only=false)
- Add .gitignore for large safetensors files
- Rewrite README with data collection, training, and inference docs
- Fix gripper PID gains and velocity limits in controller config
- Add gripper-arm synchronization state machine to inference script
- Add trajectory visualization script

File: src/ur_simulation_gz/ur_simulation_gz/urdf/ur3_ft300_robotiq_2f85.urdf.xacro (robot description, xacro)
@@ -93,5 +93,5 @@
   <link name="global_camera_mount"/>
   <joint name="global_camera_mount_joint" type="fixed">
-    <origin xyz="0 0.35 2.06" rpy="0 ${pi/2} 0"/>
+    <origin xyz="0 1.2 1.5" rpy="0 ${pi/7} -${pi/2}"/>
     <parent link="world"/>
     <child link="global_camera_mount"/>

Commit message: feat: comprehensive data pipeline overhaul + A100 V5 training guide
Data pipeline fixes (2026-06-23):
- Launch: parameter_bridge → ros_gz_image/image_bridge (lossless binary image transport)
- URDF: camera update_rate 30→50Hz
- Record: INTER_AREA resize, --hz direct recording, --start_episode resume, skip_home=false
- Record: save block/bowl positions in npz for reproducibility
- Convert: auto-skip _failed episodes
- make_video: fix default data paths

SA-MOE improvements:
- Peg-in-hole scripts synced with same fixes
- SA-MOE V8 diagnosis: dim mismatch (1024 config vs 2048 weights), alpha collapse
- Action Expert projections unfrozen for SA-MOE training

Docs:
- PROJECT_REFERENCE.md: Part 6 changelog, SA-MOE diagnosis
- README.md: updated commands, Known Issues
- A100_V5_TRAINING_GUIDE.md: Pi0 V5 full fine-tune guide

File: src/ur_simulation_gz/ur_simulation_gz/urdf/ur3_ft300_robotiq_2f85.urdf.xacro (robot description, xacro)
@@ -86,5 +86,5 @@
   <!-- ================================================================ -->
   <xacro:sensor_d435i parent="$(arg tf_prefix)wrist_3_link" name="wrist_camera" use_nominal_extrinsics="true">
-    <origin xyz="0.08 0 0" rpy="0 -${pi/3} ${pi}"/>
+    <origin xyz="0.08 0.025 -0.02" rpy="0 -${pi/2.5} ${pi}"/>
   </xacro:sensor_d435i>
   <!-- ================================================================ -->
@@ -93,5 +93,5 @@
   <link name="global_camera_mount"/>
   <joint name="global_camera_mount_joint" type="fixed">
-    <origin xyz="0 1.2 1.5" rpy="0 ${pi/7} -${pi/2}"/>
+    <origin xyz="-0.04 1.0 1.4" rpy="0 ${pi/5} -${pi/2}"/>
     <parent link="world"/>
     <child link="global_camera_mount"/>
@@ -107,11 +107,11 @@
     <sensor type="camera" name="wrist_camera_sensor">
       <always_on>1</always_on>
-      <update_rate>30</update_rate>
+      <update_rate>50</update_rate>
       <pose>0 0.015 0 0 0 0</pose>
       <camera>
         <horizontal_fov>1.210</horizontal_fov>
         <image>
-          <width>224</width>
-          <height>224</height>
+          <width>640</width>
+          <height>480</height>
           <format>R8G8B8</format>
         </image>
@@ -127,11 +127,11 @@
     <sensor type="camera" name="global_camera_sensor">
       <always_on>1</always_on>
-      <update_rate>30</update_rate>
+      <update_rate>50</update_rate>
       <pose>0 0.015 0 0 0 0</pose>
       <camera>
         <horizontal_fov>1.134</horizontal_fov>
         <image>
-          <width>224</width>
-          <height>224</height>
+          <width>640</width>
+          <height>480</height>
           <format>R8G8B8</format>
         </image>
